File: main-pcb/2v5_vccio.kicad_sch (KiCad schematic)
At the start: 11 parts, among them J8 CONN_DUMPTRUCK_HOST, U1 XC7S100-1FGGA484C, U27 NCP45525IMNTWG-H, U28 INA230

Commit message: 1088 unrouted
Connections:
- net DUT_GPIO0: now also U1.F8 (IO_L9N_T1_DQS_36); no longer U1.E8 (IO_0_36)
- net DUT_GPIO1: now also U1.G7 (IO_L11P_T1_SRCC_36); no longer U1.B9 (IO_L1P_T0_36)
- net DUT_GPIO10: now also U1.C6 (IO_L7P_T1_36); no longer U1.B7 (IO_L5N_T0_36)
- net DUT_GPIO11: now also U1.E4 (IO_L20P_T3_36); no longer U1.D8 (IO_L6P_T0_36)
- net DUT_GPIO13: now also U1.E5 (IO_L10N_T1_36); no longer U1.C6 (IO_L7P_T1_36)
- net DUT_GPIO14: now also U1.D8 (IO_L6P_T0_36); no longer U1.C5 (IO_L7N_T1_36)
- net DUT_GPIO15: now also U1.D4 (IO_L20N_T3_36); no longer U1.D6 (IO_L8P_T1_36)
- net DUT_GPIO16: now also U1.C8 (IO_L3N_T0_DQS_36); no longer U1.D5 (IO_L8N_T1_36)
- net DUT_GPIO17: now also U1.D5 (IO_L8N_T1_36); no longer U1.G8 (IO_L9P_T1_DQS_36)
- net DUT_GPIO18: now also U1.E8 (IO_0_36); no longer U1.F8 (IO_L9N_T1_DQS_36)
- net DUT_GPIO2: now also U1.F7 (IO_L12P_T1_MRCC_36); no longer U1.A9 (IO_L1N_T0_36)
- net DUT_GPIO20: now also U1.C9 (IO_L3P_T0_DQS_36); no longer U1.E5 (IO_L10N_T1_36)
- net DUT_GPIO21: now also U1.A3 (IO_L14N_T2_SRCC_36); no longer U1.G7 (IO_L11P_T1_SRCC_36)
- net DUT_GPIO22: now also U1.C3 (IO_L16N_T2_36); no longer U1.G6 (IO_L11N_T1_SRCC_36)
- net DUT_GPIO23: now also U1.B3 (IO_L15P_T2_DQS_36); no longer U1.F7 (IO_L12P_T1_MRCC_36)
- net DUT_GPIO24: now also U1.A4 (IO_L14P_T2_SRCC_36); no longer U1.F6 (IO_L12N_T1_MRCC_36)
- net DUT_GPIO25: now also U1.A2 (IO_L15N_T2_DQS_36); no longer U1.B6 (IO_L13P_T2_MRCC_36)
- net DUT_GPIO26: now also U1.C4 (IO_L16P_T2_36); no longer U1.A5 (IO_L13N_T2_MRCC_36)
- net DUT_GPIO27: now also U1.G1 (IO_L22N_T3_36); no longer U1.A4 (IO_L14P_T2_SRCC_36)
- net DUT_GPIO28: now also U1.A5 (IO_L13N_T2_MRCC_36); no longer U1.A3 (IO_L14N_T2_SRCC_36)
- net DUT_GPIO29: now also U1.G2 (IO_L22P_T3_36); no longer U1.B3 (IO_L15P_T2_DQS_36)
- net DUT_GPIO3: now also U1.G6 (IO_L11N_T1_SRCC_36); no longer U1.B10 (IO_L2P_T0_36)
- net DUT_GPIO30: now also U1.B10 (IO_L2P_T0_36); no longer U1.A2 (IO_L15N_T2_DQS_36)
- net DUT_GPIO31: now also U1.F1 (IO_L21P_T3_DQS_36); no longer U1.C4 (IO_L16P_T2_36)
- net DUT_GPIO32: now also U1.A10 (IO_L2N_T0_36); no longer U1.C3 (IO_L16N_T2_36)
- net DUT_GPIO33: now also U1.E2 (IO_L24P_T3_36); no longer U1.B2 (IO_L17P_T2_36)
- net DUT_GPIO34: now also U1.B9 (IO_L1P_T0_36); no longer U1.B1 (IO_L17N_T2_36)
- net DUT_GPIO35: now also U1.E1 (IO_L21N_T3_DQS_36); no longer U1.C2 (IO_L18P_T2_36)
- net DUT_GPIO36: now also U1.A9 (IO_L1N_T0_36); no longer U1.C1 (IO_L18N_T2_36)
- net DUT_GPIO37: now also U1.E3 (IO_L23P_T3_36); no longer U1.G4 (IO_L19P_T3_36)
- net DUT_GPIO38: now also U1.B8 (IO_L5P_T0_36); no longer U1.G3 (IO_L19N_T3_VREF_36)
- net DUT_GPIO39: now also U1.D1 (IO_L24N_T3_36); no longer U1.E4 (IO_L20P_T3_36)
- net DUT_GPIO4: now also U1.F6 (IO_L12N_T1_MRCC_36); no longer U1.A10 (IO_L2N_T0_36)
- net DUT_GPIO40: now also U1.B7 (IO_L5N_T0_36); no longer U1.D4 (IO_L20N_T3_36)
- net DUT_GPIO41: now also U1.D2 (IO_L23N_T3_36); no longer U1.F1 (IO_L21P_T3_DQS_36)
- net DUT_GPIO42: now also U1.A7 (IO_L4P_T0_36); no longer U1.E1 (IO_L21N_T3_DQS_36)
- net DUT_GPIO43: now also U1.C1 (IO_L18N_T2_36); no longer U1.G2 (IO_L22P_T3_36)
- net DUT_GPIO44: now also U1.B6 (IO_L13P_T2_MRCC_36); no longer U1.G1 (IO_L22N_T3_36)
- net DUT_GPIO45: now also U1.C2 (IO_L18P_T2_36); no longer U1.E3 (IO_L23P_T3_36)
- net DUT_GPIO46: now also U1.A6 (IO_L4N_T0_36); no longer U1.D2 (IO_L23N_T3_36)
- net DUT_GPIO47: now also U1.B1 (IO_L17N_T2_36); no longer U1.E2 (IO_L24P_T3_36)
- net DUT_GPIO48: now also U1.C5 (IO_L7N_T1_36); no longer U1.D1 (IO_L24N_T3_36)
- net DUT_GPIO49: now also U1.B2 (IO_L17P_T2_36); no longer U1.F4 (IO_25_36)
- net DUT_GPIO5: now also U1.G3 (IO_L19N_T3_VREF_36); no longer U1.C9 (IO_L3P_T0_DQS_36)
- net DUT_GPIO6: now also U1.G8 (IO_L9P_T1_DQS_36); no longer U1.C8 (IO_L3N_T0_DQS_36)
- net DUT_GPIO7: now also U1.G4 (IO_L19P_T3_36); no longer U1.A7 (IO_L4P_T0_36)
- net DUT_GPIO8: now also U1.D6 (IO_L8P_T1_36); no longer U1.A6 (IO_L4N_T0_36)
- net DUT_GPIO9: now also U1.F4 (IO_25_36); no longer U1.B8 (IO_L5P_T0_36)
Changed lines of the file:
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@@
 	)
 	(label "DUT_GPIO16"
-		(at 46.99 59.69 180)
+		(at 46.99 34.29 180)
 		(fields_autoplaced yes)
 		(effects
@@
 	)
 	(label "DUT_GPIO26"
-		(at 46.99 85.09 180)
+		(at 46.99 97.79 180)
 		(fields_autoplaced yes)
 		(effects
@@
 	)
 	(label "DUT_GPIO23"
-		(at 46.99 77.47 180)
+		(at 46.99 92.71 180)
 		(fields_autoplaced yes)
 		(effects
@@
 	)
 	(label "DUT_GPIO1"
-		(at 46.99 21.59 180)
+		(at 46.99 72.39 180)
 		(fields_autoplaced yes)
 		(effects
@@
 	)
 	(label "DUT_GPIO28"
-		(at 46.99 90.17 180)
+		(at 46.99 85.09 180)
 		(fields_autoplaced yes)
 		(effects
@@
 	)
 	(label "DUT_GPIO21"
-		(at 46.99 72.39 180)
+		(at 46.99 90.17 180)
 		(fields_autoplaced yes)
 		(effects
@@
 	)
 	(label "DUT_GPIO39"
-		(at 46.99 118.11 180)
+		(at 46.99 140.97 180)
 		(fields_autoplaced yes)
 		(effects
@@
 	)
 	(label "DUT_GPIO44"
-		(at 46.99 130.81 180)
+		(at 46.99 82.55 180)
 		(fields_autoplaced yes)
 		(effects
@@
 	)
 	(label "DUT_GPIO17"
-		(at 46.99 62.23 180)
+		(at 46.99 59.69 180)
 		(fields_autoplaced yes)
 		(effects
@@
 	)
 	(label "DUT_GPIO33"
-		(at 46.99 102.87 180)
+		(at 46.99 138.43 180)
 		(fields_autoplaced yes)
 		(effects
@@
 	)
 	(label "DUT_GPIO25"
-		(at 46.99 82.55 180)
+		(at 46.99 95.25 180)
 		(fields_autoplaced yes)
 		(effects
@@
 	)
 	(label "DUT_GPIO6"
-		(at 46.99 34.29 180)
+		(at 46.99 62.23 180)
 		(fields_autoplaced yes)
 		(effects
@@
 	)
 	(label "DUT_GPIO46"
-		(at 46.99 135.89 180)
+		(at 46.99 39.37 180)
 		(fields_autoplaced yes)
 		(effects
@@
 	)
 	(label "DUT_GPIO41"
-		(at 46.99 123.19 180)
+		(at 46.99 135.89 180)
 		(fields_autoplaced yes)
 		(effects
@@
 	)
 	(label "DUT_GPIO11"
-		(at 46.99 46.99 180)
+		(at 46.99 118.11 180)
 		(fields_autoplaced yes)
 		(effects
@@
 	)
 	(label "DUT_GPIO24"
-		(at 46.99 80.01 180)
+		(at 46.99 87.63 180)
 		(fields_autoplaced yes)
 		(effects
@@
 	)
 	(label "DUT_GPIO42"
-		(at 46.99 125.73 180)
+		(at 46.99 36.83 180)
 		(fields_autoplaced yes)
 		(effects
@@
 	)
 	(label "DUT_GPIO38"
-		(at 46.99 115.57 180)
+		(at 46.99 41.91 180)
 		(fields_autoplaced yes)
 		(effects
@@
 	)
 	(label "DUT_GPIO20"
-		(at 46.99 69.85 180)
+		(at 46.99 31.75 180)
 		(fields_autoplaced yes)
 		(effects
@@
 	)
 	(label "DUT_GPIO9"
-		(at 46.99 41.91 180)
+		(at 46.99 143.51 180)
 		(fields_autoplaced yes)
 		(effects
@@
 	)
 	(label "DUT_GPIO49"
-		(at 46.99 143.51 180)
+		(at 46.99 102.87 180)
 		(fields_autoplaced yes)
 		(effects
@@
 	)
 	(label "DUT_GPIO5"
-		(at 46.99 31.75 180)
+		(at 46.99 115.57 180)
 		(fields_autoplaced yes)
 		(effects
@@
 	)
 	(label "DUT_GPIO0"
-		(at 46.99 19.05 180)
+		(at 46.99 64.77 180)
 		(fields_autoplaced yes)
 		(effects
@@
 	)
 	(label "DUT_GPIO2"
-		(at 46.99 24.13 180)
+		(at 46.99 77.47 180)
 		(fields_autoplaced yes)
 		(effects
@@
 	)
 	(label "DUT_GPIO35"
-		(at 46.99 107.95 180)
+		(at 46.99 125.73 180)
 		(fields_autoplaced yes)
 		(effects
@@
 	)
 	(label "DUT_GPIO34"
-		(at 46.99 105.41 180)
+		(at 46.99 21.59 180)
 		(fields_autoplaced yes)
 		(effects
@@
 	)
 	(label "DUT_GPIO36"
-		(at 46.99 110.49 180)
+		(at 46.99 24.13 180)
 		(fields_autoplaced yes)
 		(effects
@@
 	)
 	(label "DUT_GPIO18"
-		(at 46.99 64.77 180)
+		(at 46.99 19.05 180)
 		(fields_autoplaced yes)
 		(effects
@@
 	)
 	(label "DUT_GPIO30"
-		(at 46.99 95.25 180)
+		(at 46.99 26.67 180)
 		(fields_autoplaced yes)
 		(effects
@@
 	)
 	(label "DUT_GPIO13"
-		(at 46.99 52.07 180)
+		(at 46.99 69.85 180)
 		(fields_autoplaced yes)
 		(effects
@@
 	)
 	(label "DUT_GPIO31"
-		(at 46.99 97.79 180)
+		(at 46.99 123.19 180)
 		(fields_autoplaced yes)
 		(effects
@@
 	)
 	(label "DUT_GPIO40"
-		(at 46.99 120.65 180)
+		(at 46.99 44.45 180)
 		(fields_autoplaced yes)
 		(effects
@@
 	)
 	(label "DUT_GPIO47"
-		(at 46.99 138.43 180)
+		(at 46.99 105.41 180)
 		(fields_autoplaced yes)
 		(effects
@@
 	)
 	(label "DUT_GPIO48"
-		(at 46.99 140.97 180)
+		(at 46.99 54.61 180)
 		(fields_autoplaced yes)
 		(effects
@@
 	)
 	(label "DUT_GPIO10"
-		(at 46.99 44.45 180)
+		(at 46.99 52.07 180)
 		(fields_autoplaced yes)
 		(effects
@@
 	)
 	(label "DUT_GPIO27"
-		(at 46.99 87.63 180)
+		(at 46.99 130.81 180)
 		(fields_autoplaced yes)
 		(effects
@@
 	)
 	(label "DUT_GPIO43"
-		(at 46.99 128.27 180)
+		(at 46.99 110.49 180)
 		(fields_autoplaced yes)
 		(effects
@@
 	)
 	(label "DUT_GPIO32"
-		(at 46.99 100.33 180)
+		(at 46.99 29.21 180)
 		(fields_autoplaced yes)
 		(effects
@@
 	)
 	(label "DUT_GPIO14"
-		(at 46.99 54.61 180)
+		(at 46.99 46.99 180)
 		(fields_autoplaced yes)
 		(effects
@@
 	)
 	(label "DUT_GPIO22"
-		(at 46.99 74.93 180)
+		(at 46.99 100.33 180)
 		(fields_autoplaced yes)
 		(effects
@@
 	)
 	(label "DUT_GPIO45"
-		(at 46.99 133.35 180)
+		(at 46.99 107.95 180)
 		(fields_autoplaced yes)
 		(effects
@@
 	)
 	(label "DUT_GPIO29"
-		(at 46.99 92.71 180)
+		(at 46.99 128.27 180)
 		(fields_autoplaced yes)
 		(effects
@@
 	)
 	(label "DUT_GPIO37"
-		(at 46.99 113.03 180)
+		(at 46.99 133.35 180)
 		(fields_autoplaced yes)
 		(effects
@@
 	)
 	(label "DUT_GPIO4"
-		(at 46.99 29.21 180)
+		(at 46.99 80.01 180)
 		(fields_autoplaced yes)
 		(effects
@@
 	)
 	(label "DUT_GPIO15"
-		(at 46.99 57.15 180)
+		(at 46.99 120.65 180)
 		(fields_autoplaced yes)
 		(effects
@@
 	)
 	(label "DUT_GPIO7"
-		(at 46.99 36.83 180)
+		(at 46.99 113.03 180)
 		(fields_autoplaced yes)
 		(effects
@@
 	)
 	(label "DUT_GPIO8"
-		(at 46.99 39.37 180)
+		(at 46.99 57.15 180)
 		(fields_autoplaced yes)
 		(effects
@@
 	)
 	(label "DUT_GPIO3"
-		(at 46.99 26.67 180)
-		(fields_autoplaced yes)
-		(effects
+		(at 46.99 74.93 180)
+		(fields_autoplaced yes)
+		(effects

Commit message: Continued routing
Connections:
- net DUT_GPIO0: now also U1.G8 (IO_L9P_T1_DQS_36); no longer U1.F8 (IO_L9N_T1_DQS_36)
- net DUT_GPIO2: now also U1.F6 (IO_L12N_T1_MRCC_36); no longer U1.F7 (IO_L12P_T1_MRCC_36)
- net DUT_GPIO4: now also U1.F7 (IO_L12P_T1_MRCC_36); no longer U1.F6 (IO_L12N_T1_MRCC_36)
- net DUT_GPIO6: now also U1.F8 (IO_L9N_T1_DQS_36); no longer U1.G8 (IO_L9P_T1_DQS_36)
Changed lines of the file:
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@@
 	)
 	(label "DUT_GPIO6"
-		(at 46.99 62.23 180)
+		(at 46.99 64.77 180)
 		(fields_autoplaced yes)
 		(effects
@@
 	)
 	(label "DUT_GPIO0"
-		(at 46.99 64.77 180)
+		(at 46.99 62.23 180)
 		(fields_autoplaced yes)
 		(effects
@@
 	)
 	(label "DUT_GPIO2"
-		(at 46.99 77.47 180)
+		(at 46.99 80.01 180)
 		(fields_autoplaced yes)
 		(effects
@@
 	)
 	(label "DUT_GPIO4"
-		(at 46.99 80.01 180)
-		(fields_autoplaced yes)
-		(effects
+		(at 46.99 77.47 180)
+		(fields_autoplaced yes)
+		(effects
