File: dut-breakouts/parallel-nor-csp56/parallel-nor-csp56.kicad_pcb (KiCad board)
At the start: 4 copper layers, 57 x 31 mm, 14 parts, among them J1 CONN_DUMPTRUCK_DEVICE, M1 LOGO, M2 LOGO, M3 LOGO, M4 LOGO, U1 MX29GL512FLXGI, U2 M24C02-RMC6TG

Commit message: parallel-nor-csp56: fixed eeprom address
Connections:
- U2 pad 1: /GND -> /3V3_EEPROM
Routing:
- net /3V3_EEPROM: track 15.3 -> 18.6 mm
- net /GND: track 125.6 -> 125.1 mm
Other:
- board text added: "DUMPTRUCK to CFI NOR CSP56 A. Zonenberg v0.2 / 2024-11-30"
- board text removed: "DUMPTRUCK to CFI NOR CSP56 A. Zonenberg v0.1 / 2024-11-20"
Changed lines of the file:
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@@
 		)
 		(property "Value" "4.7 uF"
-			(at 0 3 270)
+			(at 0 3 -90)
 			(layer "F.SilkS")
 			(hide yes)
@@
 		)
 		(property "Value" "10K"
-			(at 0 3.5 270)
+			(at 0 3.5 -90)
 			(layer "F.SilkS")
 			(hide yes)
@@
 		)
 		(property "Value" "1K"
-			(at 0 3.5 270)
+			(at 0 3.5 -90)
 			(layer "F.SilkS")
 			(hide yes)
@@
 		)
 		(property "Value" "0.47 uF"
-			(at 0.05 -3.1 360)
+			(at 0.05 -3.1 0)
 			(layer "B.SilkS")
 			(hide yes)
@@
 		)
 		(property "Value" "M24C02-RMC6TG"
-			(at -3.75 1.1 270)
+			(at -3.75 1.1 -90)
 			(layer "B.SilkS")
 			(hide yes)
@@
 			(size 0.25 0.6)
 			(layers "B.Cu" "B.Paste" "B.Mask")
-			(net 1 "/GND")
+			(net 2 "/3V3_EEPROM")
 			(pinfunction "A0")
 			(pintype "input")
@@
 		)
 		(property "Value" "0.47 uF"
-			(at 0.05 -3.1 270)
+			(at 0.05 -3.1 -90)
 			(layer "B.SilkS")
 			(hide yes)
@@
 		(layer "Edge.Cuts")
 	)
-	(gr_text "DUMPTRUCK to CFI NOR CSP56\nA. Zonenberg\nv0.1 / 2024-11-20"
+	(gr_text "DUMPTRUCK to CFI NOR CSP56\nA. Zonenberg\nv0.2 / 2024-11-30"
 		(at 35 61 0)
 		(layer "F.SilkS")
@@
 	)
 	(segment
-		(start 55.8 72.6)
-		(end 55.8 73.8935)
+		(start 53.35 76.499999)
+		(end 53.35 77.5)
 		(width 0.125)
 		(layer "B.Cu")
@@
 	)
 	(segment
-		(start 54.2 72.6)
-		(end 54.2 73.8935)
+		(start 55.8 72.6)
+		(end 55.8 73.8935)
 		(width 0.125)
 		(layer "B.Cu")
@@
 	)
 	(segment
-		(start 53.35 78.000001)
-		(end 53.35 76.499999)
-		(width 0.2)
+		(start 54.2 72.6)
+		(end 54.2 73.8935)
+		(width 0.125)
 		(layer "B.Cu")
 		(net 1)
@@
 	)
 	(segment
+		(start 56.15 78.449999)
+		(end 56.1 78.499999)
+		(width 0.125)
+		(layer "B.Cu")
+		(net 2)
+	)
+	(segment
 		(start 56.599999 74.825)
 		(end 55.6625 75.762499)
@@
 	)
 	(segment
+		(start 56.15 78.000001)
+		(end 56.15 78.449999)
+		(width 0.125)
+		(layer "B.Cu")
+		(net 2)
+	)
+	(segment
 		(start 56.6 70.2)
 		(end 56.599999 70.200001)
@@
 	(segment
 		(start 57.25 78.499999)
-		(end 56.649998 78.499999)
-		(width 0.2)
+		(end 56.1 78.499999)
+		(width 0.125)
 		(layer "B.Cu")
 		(net 2)
@@
 	)
 	(segment
-		(start 56.649998 78.499999)
-		(end 56.15 78.000001)
-		(width 0.2)
-		(layer "B.Cu")
-		(net 2)
-	)
-	(segment
 		(start 56.6 70)
 		(end 56.6 70.2)
@@
 	)
 	(segment
+		(start 56.1 78.499999)
+		(end 53.849998 78.499999)
+		(width 0.125)
+		(layer "B.Cu")
+		(net 2)
+	)
+	(segment
 		(start 57.0375 66.699999)
 		(end 57 66.737499)
@@
 		(width 0.125)
 		(layer "B.Cu")
+		(net 2)
+	)
+	(segment
+		(start 53.849998 78.499999)
+		(end 53.35 78.000001)
+		(width 0.125)
+		(layer "B.Cu")
