File: dut-breakouts/dfn8-small-qspi/dfn8-small-qspi.kicad_pcb (KiCad board)
At the start: 4 copper layers, 52.5 x 20.5 mm, 10 parts, among them J1 CONN_DUMPTRUCK_DEVICE, U1 M24C02-RMC6TG, U2 DUT_SOCKET

Commit message: dfn8-small-qspi: fixed incorrect alignment peg position
Routing:
- net /GND: vias 126 -> 127
Other:
- board text added: "DUMPTRUCK to 5x6mm DFN QSPI A. Zonenberg / v0.2 2024-12-12"
- board text removed: "DUMPTRUCK to 5x6mm DFN QSPI A. Zonenberg / v0.1 2024-12-03"
Changed lines of the file:
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@@
 				(font
 					(size 1.27 1.27)
+					(thickness 0.15)
 				)
 			)
@@
 				(font
 					(size 1.27 1.27)
+					(thickness 0.15)
 				)
 			)
@@
 				(font
 					(size 1.27 1.27)
+					(thickness 0.15)
 				)
 			)
@@
 		)
 		(pad "" np_thru_hole circle
-			(at 2.905 0)
+			(at 2.095 0)
 			(size 1.524 1.524)
 			(drill 1.125)
@@
 				(font
 					(size 1.27 1.27)
+					(thickness 0.15)
 				)
 			)
@@
 				(font
 					(size 1.27 1.27)
+					(thickness 0.15)
 				)
 			)
@@
 				(font
 					(size 1.27 1.27)
+					(thickness 0.15)
 				)
 			)
@@
 				(font
 					(size 1.27 1.27)
+					(thickness 0.15)
 				)
 			)
@@
 				(font
 					(size 1.27 1.27)
+					(thickness 0.15)
 				)
 			)
@@
 				(font
 					(size 1.27 1.27)
+					(thickness 0.15)
 				)
 			)
@@
 				(font
 					(size 1.27 1.27)
+					(thickness 0.15)
 				)
 			)
@@
 				(font
 					(size 1.27 1.27)
+					(thickness 0.15)
 				)
 			)
@@
 				(font
 					(size 1.27 1.27)
+					(thickness 0.15)
 				)
 			)
@@
 				(font
 					(size 1.27 1.27)
+					(thickness 0.15)
 				)
 			)
@@
 				(font
 					(size 1.27 1.27)
+					(thickness 0.15)
 				)
 			)
@@
 				(font
 					(size 1.27 1.27)
+					(thickness 0.15)
 				)
 			)
@@
 				(font
 					(size 1.27 1.27)
+					(thickness 0.15)
 				)
 			)
@@
 				(font
 					(size 1.27 1.27)
+					(thickness 0.15)
 				)
 			)
@@
 				(font
 					(size 1.27 1.27)
+					(thickness 0.15)
 				)
 			)
@@
 				(font
 					(size 1.27 1.27)
+					(thickness 0.15)
 				)
 			)
@@
 				(font
 					(size 1.27 1.27)
+					(thickness 0.15)
 				)
 			)
@@
 				(font
 					(size 1.27 1.27)
+					(thickness 0.15)
 				)
 			)
@@
 				(font
 					(size 1.27 1.27)
+					(thickness 0.15)
 				)
 			)
@@
 				(font
 					(size 1.27 1.27)
+					(thickness 0.15)
 				)
 			)
@@
 				(font
 					(size 1.27 1.27)
+					(thickness 0.15)
 				)
 			)
@@
 				(font
 					(size 1.27 1.27)
+					(thickness 0.15)
 				)
 				(justify mirror)
@@
 				(font
 					(size 1.27 1.27)
+					(thickness 0.15)
 				)
 				(justify mirror)
@@
 				(font
 					(size 1.27 1.27)
+					(thickness 0.15)
 				)
 				(justify mirror)
@@
 		(layer "Edge.Cuts")
 	)
-	(gr_text "DUMPTRUCK to 5x6mm DFN QSPI\nA. Zonenberg / v0.1\n2024-12-03"
+	(gr_text "DUMPTRUCK to 5x6mm DFN QSPI\nA. Zonenberg / v0.2\n2024-12-12"
 		(at 98 75 0)
 		(layer "F.SilkS")
@@
 		(size 0.45)
 		(drill 0.25)
+		(layers "F.Cu" "B.Cu")
+		(net 1)
+	)
+	(via
+		(at 72.5 72.5)
+		(size 0.45)
+		(drill 0.25)
